Commit message: Add initial control

File: description/robot_core.xacro (robot description, xacro)
@@ -21,100 +21,132 @@
         <parent link="base_link" />
         <child link="chassis"/>
-        <origin xyz ="-0.55 0 0"/>
+        <origin xyz="0 0 0.06"/>
     </joint>
     <link name="chassis">
         <visual>
-        <origin xyz="0.275 0 0.05" />
+        <origin xyz="0 0 0" />
             <geometry>
-                <box size="0.6 0.12 0.1"/>
+                <box size="0.215 0.205 0.06"/>
             </geometry>
             <material name="white"/>
         </visual>
-    </link>
-    <!-- Back chassis-->
-    <joint name="back-wheel-chassis_joint" type="fixed">
-        <parent link="chassis" />
-        <child link="back-wheel-chassis"/>
-        <origin xyz ="0 0 -0.2"/>
-    </joint>
-    <link name="back-wheel-chassis">
-        <visual>
-        <origin xyz="0 0 0.1" />
+        <collision>
+        <origin xyz="0.275 0 0.05" />
             <geometry>
-                <box size="0.1 0.12 0.2"/>
+                <box size="0.215 0.205 0.06"/>
             </geometry>
             <material name="white"/>
-        </visual>
+        </collision>
+        <xacro:inertial_box mass="0.98" x="0.215" y="0.205" z="0.06">
+            <origin xyz="0 0 0" rpy="0 0 0"/>
+        </xacro:inertial_box>
     </link>
     <!-- left back wheel link-->
     <joint name="left-back-wheel-chassis_joint" type="continuous">
-        <parent link="back-wheel-chassis" />
+        <parent link="chassis" />
         <child link="left-back-wheel-chassis"/>
-        <origin xyz ="0 0.1 0" rpy="-${pi/2} 0 0"/>
+        <origin xyz ="-0.075 0.135 -0.03" rpy="-${pi/2} 0 0"/>
         <axis xyz="0 0 1" />
     </joint>
     <link name="left-back-wheel-chassis">
+        <visual>
+        <origin xyz="0 0 0" />
+            <geometry>
+                <cylinder radius="0.03" length="0.02"/>
+            </geometry>
+        </visual>
         <collision>
         <origin xyz="0 0 0" />
             <geometry>
-                <cylinder radius="0.05" length="0.04"/>
+                <cylinder radius="0.03" length="0.02"/>
             </geometry>
         </collision>
-        <xacro:inertial_cylinder mass="0.05" length="0.04" radius="0.05">
+        <xacro:inertial_cylinder mass="0.028" length="0.02" radius="0.03">
             <origin xyz="0 0 0" rpy="0 0 0"/>
         </xacro:inertial_cylinder>
     </link>
+    <gazebo reference="left-back-wheel-chassis">
+        <material>Gazebo/Blue</material>
+    </gazebo>
     <!-- right back wheel link-->
     <joint name="right-back-wheel-chassis_joint" type="continuous">
-        <parent link="back-wheel-chassis" />
+        <parent link="chassis" />
         <child link="right-back-wheel-chassis"/>
-        <origin xyz ="0 -0.1 0" rpy="-${pi/2} 0 0"/>
+        <origin xyz ="-0.075 -0.135 -0.03" rpy="-${pi/2} 0 0"/>
         <axis xyz="0 0 1" />
     </joint>
     <link name="right-back-wheel-chassis">
+        <visual>
+        <origin xyz="0 0 0" />
+            <geometry>
+                <cylinder radius="0.03" length="0.02"/>
+            </geometry>
+        </visual>
         <collision>
         <origin xyz="0 0 0" />
             <geometry>
-                <cylinder radius="0.05" length="0.04"/>
+                <cylinder radius="0.03" length="0.02"/>
             </geometry>
         </collision>
-        <xacro:inertial_cylinder mass="0.05" length="0.04" radius="0.05">
+        <xacro:inertial_cylinder mass="0.028" length="0.02" radius="0.03">
             <origin xyz="0 0 0" rpy="0 0 0"/>
         </xacro:inertial_cylinder>
     </link>
-    <!-- Front Wheel Link-->
-    <joint name="fork-chassis-joint" type="revolute">
-        <parent link="base_link" />
-        <child link="front-wheel-driver-link" />
-        <origin xyz="0 0 0.05" />
-        <axis xyz="0 0 1" />
-        <limit lower="-0.524" upper="0.524" effort="1" velocity="0.2"/>
-    </joint>
-    <link name="front-wheel-driver-link">
-        <visual>
-        <origin xyz="0.05 0 -0.125" rpy="0 -0.5 0"/>
-            <geometry>
-                <cylinder radius="0.05" length="0.25" />
-            </geometry>
-            <material name="white"/>
-        </visual>
-    </link>
-    <!-- Front Wheel Fork -->
-    <joint name="front-wheel-joint" type="fixed">
-        <parent link="front-wheel-driver-link" />
-        <child link="front-wheel-fork"/>
-        <origin xyz ="0.125 0 -0.25" rpy="${-pi/2} 0.5 0"/>
+    <gazebo reference="right-back-wheel-chassis">
+        <material>Gazebo/Blue</material>
+    </gazebo>
+    <!-- left front wheel link-->
+    <joint name="left-front-wheel-chassis_joint" type="continuous">
+        <parent link="chassis" />
+        <child link="left-front-wheel-chassis"/>
+        <origin xyz ="0.075 0.135 -0.03" rpy="-${pi/2} 0 0"/>
         <axis xyz="0 0 1" />
     </joint>
-    <link name="front-wheel-fork">
+    <link name="left-front-wheel-chassis">
+        <visual>
+        <origin xyz="0 0 0" />
+            <geometry>
+                <cylinder radius="0.03" length="0.02"/>
+            </geometry>
+        </visual>
         <collision>
         <origin xyz="0 0 0" />
             <geometry>
-                <sphere radius="0.05"/>
+                <cylinder radius="0.03" length="0.02"/>
             </geometry>
         </collision>
-        <xacro:inertial_sphere mass="0.05" radius="0.05">
+        <xacro:inertial_cylinder mass="0.028" length="0.02" radius="0.03">
             <origin xyz="0 0 0" rpy="0 0 0"/>
-        </xacro:inertial_sphere>
+        </xacro:inertial_cylinder>
     </link>
+    <gazebo reference="left-front-wheel-chassis">
+        <material>Gazebo/Blue</material>
+    </gazebo>
+    <!-- right front wheel link-->
+    <joint name="right-front-wheel-chassis_joint" type="continuous">
+        <parent link="chassis" />
+        <child link="right-front-wheel-chassis"/>
+        <origin xyz ="0.075 -0.135 -0.03" rpy="-${pi/2} 0 0"/>
+        <axis xyz="0 0 1" />
+    </joint>
+    <link name="right-front-wheel-chassis">
+        <visual>
+        <origin xyz="0 0 0" />
+            <geometry>
+                <cylinder radius="0.03" length="0.02"/>
+            </geometry>
+        </visual>
+        <collision>
+        <origin xyz="0 0 0" />
+            <geometry>
+                <cylinder radius="0.03" length="0.02"/>
+            </geometry>
+        </collision>
+        <xacro:inertial_cylinder mass="0.028" length="0.02" radius="0.03">
+            <origin xyz="0 0 0" rpy="0 0 0"/>
+        </xacro:inertial_cylinder>
+    </link>
+    <gazebo reference="right-front-wheel-chassis">
+        <material>Gazebo/Blue</material>
+    </gazebo>
 </robot>
