Commit message: Last point of using plugin controller

File: description/gazebo_control.xacro (robot description, xacro)
@@ -3,8 +3,17 @@
      <gazebo>
         <plugin name="gz::sim::systems::DiffDrive" filename="gz-sim-diff-drive-system">
+        <ros>
+            <namespace>/</namespace>
+            <argument>--ros-args --remap cmd_vel:=cmd_vel</argument>
+            <argument>--ros-diff drive controllros2 jazzy diff drive tuWe've beenargs --remap odom:=odom</argument>
+            <update_rate>10.0</update_rate>
+        </ros>
+        <publish_odom>true</publish_odom>
+        <publish_odom_tf>true</publish_odom_tf>
+        <publish_wheel_transform>true</publish_wheel_transform>
         <!-- WHeel info-->
-        <!-- <left_joint>left-front-wheel-chassis_joint</left_joint> -->
+        <left_joint>left-front-wheel-chassis_joint</left_joint>
         <left_joint>left-back-wheel-chassis_joint</left_joint>
-        <!-- <right_joint>right-front-wheel-chassis_joint</right_joint> -->
+        <right_joint>right-front-wheel-chassis_joint</right_joint>
         <right_joint>right-back-wheel-chassis_joint</right_joint>
         <wheel_seperation>0.027</wheel_seperation>
@@ -12,9 +21,14 @@
         <max_wheel_torque>200</max_wheel_torque>
         <max_wheel_acceleration>10.0</max_wheel_acceleration>
+        <child_frame_id>base_link</child_frame_id>
         <odometry_frame>odom</odometry_frame>
         <robot_base_frame>base_link</robot_base_frame>
-        <publish_odom>true</publish_odom>
-        <publish_odom_tf>true</publish_odom_tf>
-        <publish_wheel_transform>true</publish_wheel_transform>
+        </plugin>
+        <plugin filename="gz-sim-joint-state-publisher-system" name="gz::sim::systems::JointStatePublisher">
+            <topic>joint_states</topic>
+            <joint_name>left-front-wheel-chassis_joint</joint_name>
+            <joint_name>right-front-wheel-chassis_joint</joint_name>
+            <joint_name>left-back-wheel-chassis_joint</joint_name>
+            <joint_name>right-back-wheel-chassis_joint</joint_name>
         </plugin>
     </gazebo>

File: description/robot_core.xacro (robot description, xacro)
@@ -32,5 +32,5 @@
         </visual>
         <collision>
-        <origin xyz="0.275 0 0.05" />
+        <origin xyz="0 0 0" />
             <geometry>
                 <box size="0.215 0.205 0.06"/>

Commit message: Updated URDF to match the robot's exact dimensions / weight

File: description/gazebo_control.xacro (robot description, xacro)
@@ -3,13 +3,4 @@
      <gazebo>
         <plugin name="gz::sim::systems::DiffDrive" filename="gz-sim-diff-drive-system">
-        <ros>
-            <namespace>/</namespace>
-            <argument>--ros-args --remap cmd_vel:=cmd_vel</argument>
-            <argument>--ros-diff drive controllros2 jazzy diff drive tuWe've beenargs --remap odom:=odom</argument>
-            <update_rate>10.0</update_rate>
-        </ros>
-        <publish_odom>true</publish_odom>
-        <publish_odom_tf>true</publish_odom_tf>
-        <publish_wheel_transform>true</publish_wheel_transform>
         <!-- WHeel info-->
         <left_joint>left-front-wheel-chassis_joint</left_joint>
@@ -18,16 +9,21 @@
         <right_joint>right-back-wheel-chassis_joint</right_joint>
         <wheel_seperation>0.027</wheel_seperation>
-        <wheel_diameter>0.06</wheel_diameter>
-        <max_wheel_torque>200</max_wheel_torque>
+        <wheel_radius>0.03</wheel_radius>
         <max_wheel_acceleration>10.0</max_wheel_acceleration>
+        <!-- Input -->
+        <topic>cmd_vel</topic>
+        <!-- Output -->
+        <frame_id>odom</frame_id>
         <child_frame_id>base_link</child_frame_id>
-        <odometry_frame>odom</odometry_frame>
-        <robot_base_frame>base_link</robot_base_frame>
+        <odom_topic>odom</odom_topic>
+        <odom_publisher_frequency>30</odom_publisher_frequency>
+        <tf_topic>/tf</tf_topic>
         </plugin>
-        <plugin filename="gz-sim-joint-state-publisher-system" name="gz::sim::systems::JointStatePublisher">
+        <plugin filename="gz-sim-joint-state-publisher-system"
+            name="gz::sim::systems::JointStatePublisher">
             <topic>joint_states</topic>
             <joint_name>left-front-wheel-chassis_joint</joint_name>
+            <joint_name>left-back-wheel-chassis_joint</joint_name>
             <joint_name>right-front-wheel-chassis_joint</joint_name>
-            <joint_name>left-back-wheel-chassis_joint</joint_name>
             <joint_name>right-back-wheel-chassis_joint</joint_name>
         </plugin>

File: description/robot_core.xacro (robot description, xacro)
@@ -5,12 +5,15 @@
         <color rgba="1 1 1 1" />
     </material>
-        <material name="orange">
+    <material name="orange">
         <color rgba="1 0.3 0.1 1" />
     </material>
-        <material name="blue">
+    <material name="blue">
         <color rgba="0.2 0.2 1 1" />
     </material>
-        <material name="black">
+    <material name="black">
         <color rgba="0 0 0 1" />
+    </material>
+    <material name="red">
+        <color rgba="1 0 0 1" />
     </material>
     <!-- Base Link -->
@@ -21,5 +24,5 @@
         <parent link="base_link" />
         <child link="chassis"/>
-        <origin xyz="0 0 0.06"/>
+        <origin xyz="0 0 0.0325"/>
     </joint>
     <link name="chassis">
@@ -27,12 +30,12 @@
         <origin xyz="0 0 0" />
             <geometry>
-                <box size="0.215 0.205 0.06"/>
-            </geometry>
-            <material name="white"/>
-        </visual>
-        <collision>
-        <origin xyz="0 0 0" />
-            <geometry>
-                <box size="0.215 0.205 0.06"/>
+                <box size="0.23 0.23 0.025"/>
+            </geometry>
+            <material name="white"/>
+        </visual>
+        <collision>
+        <origin xyz="0 0 0" />
+            <geometry>
+                <box size="0.23 0.23 0.025"/>
             </geometry>
             <material name="white"/>
@@ -44,34 +47,83 @@
     <!-- left back wheel link-->
     <joint name="left-back-wheel-chassis_joint" type="continuous">
+        <parent link="base_link" />
+        <child link="left-back-wheel-chassis"/>
+        <origin xyz ="-0.075 0.135 0.03" rpy="-${pi/2} 0 0"/>
+        <axis xyz="0 0 1" />
+    </joint>
+    <link name="left-back-wheel-chassis">
+        <visual>
+        <origin xyz="0 0 0" />
+            <geometry>
+                <cylinder radius="0.03" length="0.02"/>
+            </geometry>
+        </visual>
+        <collision>
+        <origin xyz="0 0 0" />
+            <geometry>
+                <cylinder radius="0.03" length="0.02"/>
+            </geometry>
+        </collision>
+        <xacro:inertial_cylinder mass="0.028" length="0.02" radius="0.03">
+            <origin xyz="0 0 0" rpy="0 0 0"/>
+        </xacro:inertial_cylinder>
+    </link>
+    <gazebo reference="left-back-wheel-chassis">
+        <material>Gazebo/Blue</material>
+    </gazebo>
+    <!-- Lidar platform-->
+    <joint name="lidar-platform-joint" type="fixed">
         <parent link="chassis" />
-        <child link="left-back-wheel-chassis"/>
-        <origin xyz ="-0.075 0.135 -0.03" rpy="-${pi/2} 0 0"/>
-        <axis xyz="0 0 1" />
-    </joint>
-    <link name="left-back-wheel-chassis">
-        <visual>
-        <origin xyz="0 0 0" />
-            <geometry>
-                <cylinder radius="0.03" length="0.02"/>
-            </geometry>
-        </visual>
-        <collision>
-        <origin xyz="0 0 0" />
-            <geometry>
-                <cylinder radius="0.03" length="0.02"/>
-            </geometry>
-        </collision>
-        <xacro:inertial_cylinder mass="0.028" length="0.02" radius="0.03">
-            <origin xyz="0 0 0" rpy="0 0 0"/>
-        </xacro:inertial_cylinder>
-    </link>
-    <gazebo reference="left-back-wheel-chassis">
-        <material>Gazebo/Blue</material>
-    </gazebo>
+        <child link="lidar-platform"/>
+        <origin xyz="0.045 0 0.036"/>
+    </joint>
+    <link name="lidar-platform">
+        <visual>
+        <origin xyz="0 0 0" />
+            <geometry>
+                <box size="0.15 0.08 0.05"/>
+            </geometry>
+            <material name="white"/>
+        </visual>
+        <collision>
+        <origin xyz="0 0 0" />
+            <geometry>
+                <box size="0.15 0.08 0.05"/>
+            </geometry>
+            <material name="white"/>
+        </collision>
+        <xacro:inertial_box mass="0.3" x="0.15" y="0.08" z="0.05">
+            <origin xyz="0 0 0" rpy="0 0 0"/>
+        </xacro:inertial_box>
+    </link>
+    <joint name="brain-joint" type="fixed">
+        <parent link="chassis" />
+        <child link="brain"/>
+        <origin xyz="-0.1 0 0.036"/>
+    </joint>
+    <link name="brain">
+        <visual>
+        <origin xyz="0 0 0" />
+            <geometry>
+                <box size="0.11 0.08 0.055"/>
+            </geometry>
+            <material name="white"/>
+        </visual>
+        <collision>
+        <origin xyz="0 0 0" />
+            <geometry>
+                <box size="0.11 0.08 0.055"/>
+            </geometry>
+            <material name="white"/>
+        </collision>
+        <xacro:inertial_box mass="0.3" x="0.11" y="0.08" z="0.055">
+            <origin xyz="0 0 0" rpy="0 0 0"/>
+        </xacro:inertial_box>
+    </link>
     <!-- right back wheel link-->
     <joint name="right-back-wheel-chassis_joint" type="continuous">
-        <parent link="chassis" />
+        <parent link="base_link" />
         <child link="right-back-wheel-chassis"/>
-        <origin xyz ="-0.075 -0.135 -0.03" rpy="-${pi/2} 0 0"/>
+        <origin xyz ="-0.075 -0.135 0.03" rpy="-${pi/2} 0 0"/>
         <axis xyz="0 0 1" />
     </joint>
@@ -98,7 +150,7 @@
     <!-- left front wheel link-->
     <joint name="left-front-wheel-chassis_joint" type="continuous">
-        <parent link="chassis" />
+        <parent link="base_link" />
         <child link="left-front-wheel-chassis"/>
-        <origin xyz ="0.075 0.135 -0.03" rpy="-${pi/2} 0 0"/>
+        <origin xyz ="0.075 0.135 0.03" rpy="-${pi/2} 0 0"/>
         <axis xyz="0 0 1" />
     </joint>
@@ -125,7 +177,7 @@
     <!-- right front wheel link-->
     <joint name="right-front-wheel-chassis_joint" type="continuous">
-        <parent link="chassis" />
+        <parent link="base_link" />
         <child link="right-front-wheel-chassis"/>
-        <origin xyz ="0.075 -0.135 -0.03" rpy="-${pi/2} 0 0"/>
+        <origin xyz ="0.075 -0.135 0.03" rpy="-${pi/2} 0 0"/>
         <axis xyz="0 0 1" />
     </joint>

Commit message: Update to new gazebo

File: description/gazebo_control.xacro (robot description, xacro)
@@ -4,17 +4,27 @@
         <plugin name="gz::sim::systems::DiffDrive" filename="gz-sim-diff-drive-system">
         <!-- WHeel info-->
-        <!-- <left_joint>left-front-wheel-chassis_joint</left_joint> -->
+        <left_joint>left-front-wheel-chassis_joint</left_joint>
         <left_joint>left-back-wheel-chassis_joint</left_joint>
-        <!-- <right_joint>right-front-wheel-chassis_joint</right_joint> -->
+        <right_joint>right-front-wheel-chassis_joint</right_joint>
         <right_joint>right-back-wheel-chassis_joint</right_joint>
         <wheel_seperation>0.027</wheel_seperation>
-        <wheel_diameter>0.06</wheel_diameter>
-        <max_wheel_torque>200</max_wheel_torque>
+        <wheel_radius>0.03</wheel_radius>
         <max_wheel_acceleration>10.0</max_wheel_acceleration>
-        <odometry_frame>odom</odometry_frame>
-        <robot_base_frame>base_link</robot_base_frame>
-        <publish_odom>true</publish_odom>
-        <publish_odom_tf>true</publish_odom_tf>
-        <publish_wheel_transform>true</publish_wheel_transform>
+        <!-- Input -->
+        <topic>cmd_vel</topic>
+        <!-- Output -->
+        <frame_id>odom</frame_id>
+        <child_frame_id>base_link</child_frame_id>
+        <odom_topic>odom</odom_topic>
+        <odom_publisher_frequency>30</odom_publisher_frequency>
+        <tf_topic>/tf</tf_topic>
+        </plugin>
+        <plugin filename="gz-sim-joint-state-publisher-system"
+            name="gz::sim::systems::JointStatePublisher">
+            <topic>joint_states</topic>
+            <joint_name>left-front-wheel-chassis_joint</joint_name>
+            <joint_name>left-back-wheel-chassis_joint</joint_name>
+            <joint_name>right-front-wheel-chassis_joint</joint_name>
+            <joint_name>right-back-wheel-chassis_joint</joint_name>
         </plugin>
     </gazebo>

File: description/robot_core.xacro (robot description, xacro)
@@ -32,5 +32,5 @@
         </visual>
         <collision>
-        <origin xyz="0.275 0 0.05" />
+        <origin xyz="0 0 0" />
             <geometry>
                 <box size="0.215 0.205 0.06"/>
@@ -44,7 +44,7 @@
     <!-- left back wheel link-->
     <joint name="left-back-wheel-chassis_joint" type="continuous">
-        <parent link="chassis" />
+        <parent link="base_link" />
         <child link="left-back-wheel-chassis"/>
-        <origin xyz ="-0.075 0.135 -0.03" rpy="-${pi/2} 0 0"/>
+        <origin xyz ="-0.075 0.135 0.03" rpy="-${pi/2} 0 0"/>
         <axis xyz="0 0 1" />
     </joint>
@@ -71,7 +71,7 @@
     <!-- right back wheel link-->
     <joint name="right-back-wheel-chassis_joint" type="continuous">
-        <parent link="chassis" />
+        <parent link="base_link" />
         <child link="right-back-wheel-chassis"/>
-        <origin xyz ="-0.075 -0.135 -0.03" rpy="-${pi/2} 0 0"/>
+        <origin xyz ="-0.075 -0.135 0.03" rpy="-${pi/2} 0 0"/>
         <axis xyz="0 0 1" />
     </joint>
@@ -98,7 +98,7 @@
     <!-- left front wheel link-->
     <joint name="left-front-wheel-chassis_joint" type="continuous">
-        <parent link="chassis" />
+        <parent link="base_link" />
         <child link="left-front-wheel-chassis"/>
-        <origin xyz ="0.075 0.135 -0.03" rpy="-${pi/2} 0 0"/>
+        <origin xyz ="0.075 0.135 0.03" rpy="-${pi/2} 0 0"/>
         <axis xyz="0 0 1" />
     </joint>
@@ -125,7 +125,7 @@
     <!-- right front wheel link-->
     <joint name="right-front-wheel-chassis_joint" type="continuous">
-        <parent link="chassis" />
+        <parent link="base_link" />
         <child link="right-front-wheel-chassis"/>
-        <origin xyz ="0.075 -0.135 -0.03" rpy="-${pi/2} 0 0"/>
+        <origin xyz ="0.075 -0.135 0.03" rpy="-${pi/2} 0 0"/>
         <axis xyz="0 0 1" />
     </joint>
