Commit message: Add initial communication attempts

File: robotics-project/description/robot_core.xacro (robot description, xacro)
@@ -45,31 +45,4 @@
         </xacro:inertial_box>
     </link>
-    <!-- left back wheel link-->
-    <joint name="left-back-wheel-chassis_joint" type="continuous">
-        <parent link="base_link" />
-        <child link="left-back-wheel-chassis"/>
-        <origin xyz ="-0.075 0.135 0.03" rpy="-${pi/2} 0 0"/>
-        <axis xyz="0 0 1" />
-    </joint>
-    <link name="left-back-wheel-chassis">
-        <visual>
-        <origin xyz="0 0 0" />
-            <geometry>
-                <cylinder radius="0.03" length="0.02"/>
-            </geometry>
-        </visual>
-        <collision>
-        <origin xyz="0 0 0" />
-            <geometry>
-                <cylinder radius="0.03" length="0.02"/>
-            </geometry>
-        </collision>
-        <xacro:inertial_cylinder mass="0.028" length="0.02" radius="0.03">
-            <origin xyz="0 0 0" rpy="0 0 0"/>
-        </xacro:inertial_cylinder>
-    </link>
-    <gazebo reference="left-back-wheel-chassis">
-        <material>Gazebo/Blue</material>
-    </gazebo>
     <!-- Lidar platform-->
     <joint name="lidar-platform-joint" type="fixed">
@@ -121,4 +94,31 @@
         </xacro:inertial_box>
     </link>
+    <!-- left back wheel link-->
+    <joint name="left-back-wheel-chassis_joint" type="continuous">
+        <parent link="base_link" />
+        <child link="left-back-wheel-chassis"/>
+        <origin xyz ="-0.075 0.135 0.03" rpy="-${pi/2} 0 0"/>
+        <axis xyz="0 0 1" />
+    </joint>
+    <link name="left-back-wheel-chassis">
+        <visual>
+        <origin xyz="0 0 0" />
+            <geometry>
+                <cylinder radius="0.03" length="0.02"/>
+            </geometry>
+        </visual>
+        <collision>
+        <origin xyz="0 0 0" />
+            <geometry>
+                <cylinder radius="0.03" length="0.02"/>
+            </geometry>
+        </collision>
+        <xacro:inertial_cylinder mass="0.028" length="0.02" radius="0.03">
+            <origin xyz="0 0 0" rpy="0 0 0"/>
+        </xacro:inertial_cylinder>
+    </link>
+    <gazebo reference="left-back-wheel-chassis">
+        <material>Gazebo/Blue</material>
+    </gazebo>
     <!-- right back wheel link-->
     <joint name="right-back-wheel-chassis_joint" type="continuous">

File: robotics-project/description/robot_simulation_core.xacro (robot description, xacro)
@@ -21,5 +21,5 @@
         <parent link="base_link" />
         <child link="chassis"/>
-        <origin xyz="0 0 0.06"/>
+        <origin xyz="0 0 0.0325"/>
     </joint>
     <link name="chassis">
@@ -27,16 +27,65 @@
         <origin xyz="0 0 0" />
             <geometry>
-                <box size="0.215 0.205 0.06"/>
-            </geometry>
-            <material name="white"/>
-        </visual>
-        <collision>
-        <origin xyz="0 0 0" />
-            <geometry>
-                <box size="0.215 0.205 0.06"/>
+                <box size="0.23 0.23 0.025"/>
+            </geometry>
+            <material name="white"/>
+        </visual>
+        <collision>
+        <origin xyz="0 0 0" />
+            <geometry>
+                <box size="0.23 0.23 0.025"/>
             </geometry>
             <material name="white"/>
         </collision>
         <xacro:inertial_box mass="0.98" x="0.215" y="0.205" z="0.06">
+            <origin xyz="0 0 0" rpy="0 0 0"/>
+        </xacro:inertial_box>
+    </link>
+    <!-- Lidar platform-->
+    <joint name="lidar-platform-joint" type="fixed">
+        <parent link="chassis" />
+        <child link="lidar-platform"/>
+        <origin xyz="0.045 0 0.036"/>
+    </joint>
+    <link name="lidar-platform">
+        <visual>
+        <origin xyz="0 0 0" />
+            <geometry>
+                <box size="0.15 0.08 0.05"/>
+            </geometry>
+            <material name="white"/>
+        </visual>
+        <collision>
+        <origin xyz="0 0 0" />
+            <geometry>
+                <box size="0.15 0.08 0.05"/>
+            </geometry>
+            <material name="white"/>
+        </collision>
+        <xacro:inertial_box mass="0.3" x="0.15" y="0.08" z="0.05">
+            <origin xyz="0 0 0" rpy="0 0 0"/>
+        </xacro:inertial_box>
+    </link>
+    <joint name="brain-joint" type="fixed">
+        <parent link="chassis" />
+        <child link="brain"/>
+        <origin xyz="-0.1 0 0.03"/>
+    </joint>
+    <link name="brain">
+        <visual>
+        <origin xyz="0 0 0" />
+            <geometry>
+                <box size="0.11 0.08 0.055"/>
+            </geometry>
+            <material name="white"/>
+        </visual>
+        <collision>
+        <origin xyz="0 0 0" />
+            <geometry>
+                <box size="0.11 0.08 0.055"/>
+            </geometry>
+            <material name="white"/>
+        </collision>
+        <xacro:inertial_box mass="0.3" x="0.11" y="0.08" z="0.055">
             <origin xyz="0 0 0" rpy="0 0 0"/>
         </xacro:inertial_box>
@@ -98,7 +147,7 @@
     <!-- CASTER WHEEL FRONT LINK -->
     <joint name="caster_wheel_front_joint" type="fixed">
-        <parent link="base_link"/>
+        <parent link="chassis"/>
         <child link="caster_wheel_front"/>
-        <origin xyz="0.075 0 0.03"/>
+        <origin xyz="0.08 0 0"/>
     </joint>
     <link name="caster_wheel_front">
@@ -120,12 +169,12 @@
     <gazebo reference="caster_wheel_front">
         <material>Gazebo/White</material>
-        <mu1 value="0.001"/>
-        <mu2 value="0.001"/>
+        <mu1 value="0.00001"/>
+        <mu2 value="0.00001"/>
     </gazebo>
     <!-- CASTER WHEEL Back LINK -->
     <joint name="caster_wheel_back_joint" type="fixed">
-        <parent link="base_link"/>
+        <parent link="chassis"/>
         <child link="caster_wheel_back"/>
-        <origin xyz="-0.075 0 0.03"/>
+        <origin xyz="-0.08 0 0"/>
     </joint>
     <link name="caster_wheel_back">
@@ -147,6 +196,6 @@
     <gazebo reference="caster_wheel">
         <material>Gazebo/White</material>
-        <mu1 value="0.001"/>
-        <mu2 value="0.001"/>
+        <mu1 value="0.00001"/>
+        <mu2 value="0.00001"/>
     </gazebo>
 </robot>

File: robotics-project/description/ros2_control.xacro (robot description, xacro)
@@ -1,29 +1,61 @@
 <?xml version="1.0"?>
-<robot xmlns:xacro="http://www.ros.org/wiki/xacro">
-    <ros2_control name="GazeboSystem" type="system">
-        <hardware>
-            <plugin>gz_ros2_control/GazeboSimSystem</plugin>
-        </hardware>
-        <joint name="left-wheel-chassis_joint">
-            <command_interface name="velocity">
-                <param name="min">-10</param>
-                <param name="max">10</param>
-            </command_interface>
-            <state_interface name="velocity"/>
-            <state_interface name="position"/>
-        </joint>
-        <joint name="right-wheel-chassis_joint">
-            <command_interface name="velocity">
-                <param name="min">-10</param>
-                <param name="max">10</param>
-            </command_interface>
-            <state_interface name="velocity"/>
-            <state_interface name="position"/>
-        </joint>
-    </ros2_control>
-    <gazebo>
-        <plugin filename="gz_ros2_control-system" name="gz_ros2_control::GazeboSimROS2ControlPlugin">
-            <parameters>$(find robotics-project)/config/my_controllers.yaml</parameters>
-        </plugin>
-    </gazebo>
-</robot>
+ <robot xmlns:xacro="http://www.ros.org/wiki/xacro">
+    <xacro:unless value="$(arg sim_mode)">
+        <ros2_control name="RealRobot" type="system">
+            <hardware>
+                <plugin>vex_control/VexHardware</plugin>
+                <param name="left_wheel_name">left-wheel-chassis_joint</param>
+                <param name="right_wheel_name">right-wheel-chassis_joint</param>
+                <param name="loop_rate">30</param>
+                <param name="device">/dev/ttyACM1</param>
+                <param name="baud_rate">115200</param>
+                <param name="timeout_ms">3000</param>
+                <param name="enc_counts_per_rev">360</param>
+            </hardware>
+            <joint name="left-wheel-chassis_joint">
+                <command_interface name="velocity">
+                    <param name="min">-10</param>
+                    <param name="max">10</param>
+                </command_interface>
+                <state_interface name="position"/>
+                <state_interface name="velocity"/>
+            </joint>
+            <joint name="right-wheel-chassis_joint">
+                <command_interface name="velocity">
+                    <param name="min">-10</param>
+                    <param name="max">10</param>
+                </command_interface>
+                <state_interface name="position"/>
+                <state_interface name="velocity"/>
+            </joint>
+        </ros2_control>
+    </xacro:unless>
+    <xacro:if value="$(arg sim_mode)">
+     <ros2_control name="GazeboSystem" type="system">
+         <hardware>
+             <plugin>gz_ros2_control/GazeboSimSystem</plugin>
+         </hardware>
+         <joint name="left-wheel-chassis_joint">
+             <command_interface name="velocity">
+                 <param name="min">-10</param>
+                 <param name="max">10</param>
+             </command_interface>
+             <state_interface name="velocity"/>
+             <state_interface name="position"/>
+         </joint>
+         <joint name="right-wheel-chassis_joint">
+             <command_interface name="velocity">
+                 <param name="min">-10</param>
+                 <param name="max">10</param>
+             </command_interface>
+             <state_interface name="velocity"/>
+             <state_interface name="position"/>
+         </joint>
+     </ros2_control>
+     <gazebo>
+         <plugin filename="gz_ros2_control-system" name="gz_ros2_control::GazeboSimROS2ControlPlugin">
+             <parameters>$(find robotics-project)/config/my_controllers.yaml</parameters>
+         </plugin>
+     </gazebo>
+     </xacro:if>
+ </robot>
