Commit message: Get real robot working and rplidar launch file

File: robotics-project/description/lidar.xacro (robot description, xacro)
@@ -4,5 +4,5 @@
         <parent link="chassis"/>
         <child link="laser_frame"/>
-        <origin xyz="0 0 0.082" rpy="0 0 0"/>
+        <origin xyz="0 0 0.082" rpy="0 0 ${pi/2}"/>
     </joint>
     <link name="laser_frame">

File: robotics-project/description/ros2_control.xacro (robot description, xacro)
@@ -11,10 +11,10 @@
                 <param name="baud_rate">115200</param>
                 <param name="timeout_ms">3000</param>
-                <param name="enc_counts_per_rev">360</param>
+                <param name="enc_counts_per_rev">900</param>
             </hardware>
             <joint name="left-wheel-chassis_joint">
                 <command_interface name="velocity">
-                    <param name="min">-10</param>
-                    <param name="max">10</param>
+                    <param name="min">-1</param>
+                    <param name="max">1</param>
                 </command_interface>
                 <state_interface name="position"/>
@@ -23,6 +23,6 @@
             <joint name="right-wheel-chassis_joint">
                 <command_interface name="velocity">
-                    <param name="min">-10</param>
-                    <param name="max">10</param>
+                    <param name="min">-1</param>
+                    <param name="max">1</param>
                 </command_interface>
                 <state_interface name="position"/>

Commit message: Ensure lidar working and begin adding slam toolbox stuff

File: robotics-project/description/lidar.xacro (robot description, xacro)
@@ -13,9 +13,4 @@
             <material name="black"/>
         </visual>
-        <collision>
-            <geometry>
-                <cylinder radius="0.04" length="0.04"/>
-            </geometry>
-        </collision>
         <xacro:inertial_cylinder mass="0.4" length="0.04" radius="0.05">
             <origin xyz="0 0 0" rpy="0 0 0"/>
@@ -24,8 +19,7 @@
     <gazebo reference="laser_frame">
         <material>Gazebo/Black</material>
-        <sensor name="laser" type="lidar">
+        <sensor name="laser" type="gpu_lidar">
             <pose> 0 0 0 0 0 0 </pose>
             <visualize>true</visualize>
-            <always_on>1</always_on>
             <update_rate>10</update_rate>
             <lidar>
@@ -38,9 +32,10 @@
                 </scan>
                 <range>
-                    <min>0.3</min>
+                    <min>0.2</min>
                     <max>12</max>
                 </range>
             </lidar>
             <topic>scan</topic>
+            <gz_frame_id>laser_frame</gz_frame_id>
         </sensor>
     </gazebo>

File: robotics-project/description/robot_simulation_core.xacro (robot description, xacro)
@@ -17,4 +17,12 @@
     <link name= "base_link">
     </link>
+    <!-- Base Footprint Link -->
+    <joint name="base_footprint_joint" type="fixed">
+        <parent link="base_link" />
+        <child link="base_footprint" />
+        <origin xyz="0 0 0" rpy="0 0 0" />
+    </joint>
+    <link name= "base_footprint">
+    </link>
     <!-- Chassis Link -->
     <joint name="chassis_joint" type="fixed">
@@ -147,5 +155,5 @@
     <!-- CASTER WHEEL FRONT LINK -->
     <joint name="caster_wheel_front_joint" type="fixed">
-        <parent link="chassis"/>
+        <parent link="base_link"/>
         <child link="caster_wheel_front"/>
         <origin xyz="0.08 0 0"/>
@@ -174,5 +182,5 @@
     <!-- CASTER WHEEL Back LINK -->
     <joint name="caster_wheel_back_joint" type="fixed">
-        <parent link="chassis"/>
+        <parent link="base_link"/>
         <child link="caster_wheel_back"/>
         <origin xyz="-0.08 0 0"/>
