Commit message: Add slam toolbox params

File: robotics-project/description/robot_simulation_core.xacro (robot description, xacro)
@@ -124,4 +124,6 @@
     </link>
     <gazebo reference="left-wheel-chassis">
+        <mu1>0.2</mu1>
+        <mu2>0.2</mu2>
         <material>Gazebo/Blue</material>
     </gazebo>
@@ -151,4 +153,6 @@
     </link>
     <gazebo reference="right-wheel-chassis">
+        <mu1>0.2</mu1>
+        <mu2>0.2</mu2>
         <material>Gazebo/Blue</material>
     </gazebo>
@@ -157,5 +161,5 @@
         <parent link="base_link"/>
         <child link="caster_wheel_front"/>
-        <origin xyz="0.08 0 0"/>
+        <origin xyz="0.08 0 0.0301"/>
     </joint>
     <link name="caster_wheel_front">
@@ -184,5 +188,5 @@
         <parent link="base_link"/>
         <child link="caster_wheel_back"/>
-        <origin xyz="-0.08 0 0"/>
+        <origin xyz="-0.08 0 0.0301"/>
     </joint>
     <link name="caster_wheel_back">
@@ -202,5 +206,5 @@
         </xacro:inertial_sphere>
     </link>
-    <gazebo reference="caster_wheel">
+    <gazebo reference="caster_wheel_back">
         <material>Gazebo/White</material>
         <mu1 value="0.00001"/>
